File: Schematics/BatteryBoxEuro.sch (KiCad schematic (older format))
At the start: 16 parts, among them K1 JD2912-1Z-12VDC_40A, P1 Conn_WallPlug, U1 Terminal16, U2 F_Distributor, U3 NAC3MPA-1-WOT, U4 DPlusSimulator, U5 Pulser, U6 230V_KfzCharger, U9 NAC3MPA-1-WOT, X1 X3, X2 12VKfz_Plug, X3 X3

Commit message: finalize schematic
Parts:
- U4: renamed from U3; symbol NAC3MPA-1-WOT:NAC3MPA-1-WOT -> BatteryBox-rescue:NAC3MPA-1-WOT-NAC3MPA-1-WOT
- U6: renamed from U9; symbol NAC3MPA-1-WOT:NAC3MPA-1-WOT -> BatteryBox-rescue:NAC3MPA-1-WOT-NAC3MPA-1-WOT
- renumbered BT2 to BT1, F2 to F1, F1 to F2, U4 to U3, U1 to U5, U2 to U7, U6 to U8, U5 to U9, X1 to X3, X3 to X4
Changed lines of the file:
@@
 $EndDescr
 $Comp
-L Device:Fuse F1
+L Device:Fuse F2
 U 1 1 5E86EA9E
 P 10650 2850
-F 0 "F1" H 10710 2896 50  0000 L CNN
+F 0 "F2" H 10710 2896 50  0000 L CNN
 F 1 "50A" H 10710 2805 50  0000 L CNN
 F 2 "" V 10580 2850 50  0001 C CNN
@@
 $EndComp
 $Comp
-L Device:Battery BT2
+L Device:Battery BT1
 U 1 1 5E872FAE
 P 10650 4250
-F 0 "BT2" H 10758 4296 50  0000 L CNN
+F 0 "BT1" H 10758 4296 50  0000 L CNN
 F 1 "12V" H 10758 4205 50  0000 L CNN
 F 2 "" V 10650 4310 50  0001 C CNN
@@
 $EndComp
 $Comp
-L MyParts:DPlusSimulator U4
+L MyParts:DPlusSimulator U3
 U 1 1 5E87470E
 P 1150 3100
-F 0 "U4" H 2028 3171 50  0000 L CNN
+F 0 "U3" H 2028 3171 50  0000 L CNN
 F 1 "DPlusSimulator" H 2028 3080 50  0000 L CNN
 F 2 "" H 900 3600 50  0001 C CNN
@@
 $EndComp
 $Comp
-L MyParts:Pulser U5
+L MyParts:Pulser U9
 U 1 1 5E879508
 P 10150 3550
-F 0 "U5" V 10104 3628 50  0000 L CNN
+F 0 "U9" V 10104 3628 50  0000 L CNN
 F 1 "Pulser" V 10195 3628 50  0000 L CNN
 F 2 "" H 10150 3550 50  0001 C CNN
@@
 $EndComp
 $Comp
-L MyParts:F_Distributor U2
+L MyParts:F_Distributor U7
 U 1 1 5E8A7CC8
 P 7350 2800
-F 0 "U2" H 7350 1977 50  0000 C CNN
+F 0 "U7" H 7350 1977 50  0000 C CNN
 F 1 "F_Distributor" H 7350 1886 50  0000 C CNN
 F 2 "" H 7350 2800 50  0001 C CNN
@@
 	10050 4150 10050 5950
 $Comp
-L Connector:Conn_WallSocket X3
+L Connector:Conn_WallSocket X4
 U 1 1 5EBD0381
 P 6950 4350
-F 0 "X3" V 6906 4162 50  0000 R CNN
+F 0 "X4" V 6906 4162 50  0000 R CNN
 F 1 "X3" V 6861 4162 50  0001 R CNN
 F 2 "" H 6550 4350 50  0001 C CNN
@@
 	8100 4900 8100 4050
 $Comp
-L Device:Fuse F2
+L Device:Fuse F1
 U 1 1 5EBE1E9A
 P 7550 4250
-F 0 "F2" H 7610 4296 50  0000 L CNN
+F 0 "F1" H 7610 4296 50  0000 L CNN
 F 1 "10A" H 7610 4205 50  0000 L CNN
 F 2 "" V 7480 4250 50  0001 C CNN
@@
 12V Zigarettenanzünder\n- 1m Kabel -
 $Comp
-L MyParts:230V_KfzCharger U6
+L MyParts:230V_KfzCharger U8
 U 1 1 5EC5CF8F
 P 8650 750
-F 0 "U6" H 8850 815 50  0000 C CNN
+F 0 "U8" H 8850 815 50  0000 C CNN
 F 1 "230V_KfzCharger" H 8850 724 50  0000 C CNN
 F 2 "" H 8650 750 50  0001 C CNN
@@
 	4100 3200 6800 3200
 $Comp
-L NAC3MPA-1-WOT:NAC3MPA-1-WOT U3
+L BatteryBox-rescue:NAC3MPA-1-WOT-NAC3MPA-1-WOT U4
 U 1 1 5EF1E21B
 P 3700 1450
-F 0 "U3" V 3461 2080 50  0000 L CNN
+F 0 "U4" V 3461 2080 50  0000 L CNN
 F 1 "NAC3MPA-1-WOT" V 3552 2080 50  0000 L CNN
 F 2 "NAC3MPA-1-WOT" H 3700 1450 50  0001 L BNN
@@
 	2300 2750 2300 3700
 $Comp
-L Connector:Conn_WallSocket X1
+L Connector:Conn_WallSocket X3
 U 1 1 5EC190DC
 P 5550 4350
-F 0 "X1" V 5506 4162 50  0000 R CNN
+F 0 "X3" V 5506 4162 50  0000 R CNN
 F 1 "X3" V 5461 4162 50  0001 R CNN
 F 2 "" H 5150 4350 50  0001 C CNN
@@
 	5850 3000 6800 3000
 $Comp
-L NAC3MPA-1-WOT:NAC3MPA-1-WOT U9
+L BatteryBox-rescue:NAC3MPA-1-WOT-NAC3MPA-1-WOT U6
 U 1 1 5F024C85
 P 5450 1450
-F 0 "U9" V 5211 2080 50  0000 L CNN
+F 0 "U6" V 5211 2080 50  0000 L CNN
 F 1 "NAC3MPA-1-WOT" V 5302 2080 50  0000 L CNN
 F 2 "NAC3MPA-1-WOT" H 5450 1450 50  0001 L BNN
@@
 	5850 1650 5850 3000
 $Comp
-L MyParts:Terminal16 U1
+L MyParts:Terminal16 U5
 U 1 1 5EF240EF
 P 4900 5600
-F 0 "U1" H 5328 5646 50  0000 L CNN
+F 0 "U5" H 5328 5646 50  0000 L CNN
 F 1 "Terminal16" H 5328 5555 50  0000 L CNN
 F 2 "MyParts:GroundTerminal" H 4950 5650 50  0001 C CNN
