File: Schematics/CoolerBox.sch (KiCad schematic (older format))
At the start: 6 parts, among them J5 12VDC Kfz, J6 12VDC Kfz, SW1 S1, U7 DometicCF35, U8 USB_Charger

Commit message: finalize schematic
Parts:
- renumbered J5 to J1, J6 to J2, U8 to U1, U7 to U2
Changed lines of the file:
@@
 $EndDescr
 $Comp
-L Connector:Conn_WallSocket J5
+L Connector:Conn_WallSocket J1
 U 1 1 5EF09B1F
 P 4000 3000
-F 0 "J5" H 3956 3325 50  0000 C CNN
+F 0 "J1" H 3956 3325 50  0000 C CNN
 F 1 "12VDC Kfz" H 3956 3234 50  0000 C CNN
 F 2 "" H 3600 3000 50  0001 C CNN
@@
 $EndComp
 $Comp
-L Connector:Conn_WallSocket J6
+L Connector:Conn_WallSocket J2
 U 1 1 5EF0A29B
 P 5000 3000
-F 0 "J6" H 4956 3325 50  0000 C CNN
+F 0 "J2" H 4956 3325 50  0000 C CNN
 F 1 "12VDC Kfz" H 4956 3234 50  0000 C CNN
 F 2 "" H 4600 3000 50  0001 C CNN
@@
 AC_N
 $Comp
-L MyParts:DometicCF35 U7
+L MyParts:DometicCF35 U2
 U 1 1 5EF0EA96
 P 9000 3350
-F 0 "U7" H 9578 2821 50  0000 L CNN
+F 0 "U2" H 9578 2821 50  0000 L CNN
 F 1 "DometicCF35" H 9578 2730 50  0000 L CNN
 F 2 "" H 9000 3350 50  0001 C CNN
@@
 Connection ~ 3000 1500
 $Comp
-L MyParts:USB_Charger U8
+L MyParts:USB_Charger U1
 U 1 1 5EF0F9B5
 P 6950 2300
-F 0 "U8" H 7478 1746 50  0000 L CNN
+F 0 "U1" H 7478 1746 50  0000 L CNN
 F 1 "USB_Charger" H 7478 1655 50  0000 L CNN
 F 2 "" H 6950 2300 50  0001 C CNN
