File: Schematics/KleinVerteiler230V.sch (KiCad schematic (older format))
At the start: 3 parts

Commit message: some modifications
Parts:
- gave numbers to parts that had none: 3
Changed lines of the file:
@@
 $Descr A4 11693 8268
 encoding utf-8
-Sheet 6 6
+Sheet 4 4
 Title ""
 Date ""
@@
 $EndDescr
 $Comp
-L Relay:FINDER-30.22 K?
+L Relay:FINDER-30.22 K3
 U 1 1 5F16ADE4
 P 5800 4300
-F 0 "K?" H 6430 4346 50  0000 L CNN
+F 0 "K3" H 6430 4346 50  0000 L CNN
 F 1 "FINDER-30.22" H 6430 4255 50  0000 L CNN
 F 2 "Relay_THT:Relay_DPDT_Finder_30.22" H 7150 4270 50  0001 C CNN
@@
 $EndComp
 $Comp
-L MyParts:FI Q?
+L MyParts:FI Q1
 U 1 1 5F16CA33
 P 3900 2250
-F 0 "Q?" V 3435 2025 50  0000 C CNN
+F 0 "Q1" V 3435 2025 50  0000 C CNN
 F 1 "FI" V 3526 2025 50  0000 C CNN
 F 2 "" H 3900 2250 50  0001 C CNN
@@
 $EndComp
 $Comp
-L Device:Polyfuse F?
+L Device:Polyfuse F2
 U 1 1 5F16D2C4
 P 3450 1050
-F 0 "F?" V 3225 1050 50  0000 C CNN
+F 0 "F2" V 3225 1050 50  0000 C CNN
 F 1 "10A-B" V 3316 1050 50  0000 C CNN
 F 2 "" H 3500 850 50  0001 L CNN
@@
 Text HLabel 10550 2650 2    50   Input ~ 0
 230V_PE_OutS
+Wire Notes Line
+	1550 950  1550 1550
+Wire Notes Line
+	1550 1550 1650 1550
+Wire Notes Line
+	1650 1550 1650 950
+Wire Notes Line
+	1650 950  1550 950
+Wire Notes Line
+	1550 1950 1550 2550
+Wire Notes Line
+	1550 2550 1650 2550
+Wire Notes Line
+	1650 2550 1650 1950
+Wire Notes Line
+	1650 1950 1550 1950
+Wire Notes Line
+	10200 950  10300 950
+Wire Notes Line
+	10300 950  10300 1550
+Wire Notes Line
+	10300 1550 10200 1550
+Wire Notes Line
+	10200 1550 10200 950
+Wire Notes Line
+	10200 2150 10200 2750
+Wire Notes Line
+	10200 2750 10300 2750
+Wire Notes Line
+	10300 2750 10300 2150
+Wire Notes Line
+	10300 2150 10200 2150
 $EndSCHEMATC

Commit message: modyfy schematic regarding new concept (still in work)
Parts:
- K3: symbol Relay:FINDER-30.22 -> MyParts:FINDER-30.22
Connections:
- net 230V_L_OutS: now also K3.12; no longer K3.11
- net 230V_N: now also K3.5, K3.A2; no longer K3.22
- net 230V_N_OutS: now also K3.9; no longer K3.21
- net 230V_L_Out: no longer names the net of F2.1
- net 230V_L_Out: now also K3.8, K3.A1; no longer K3.12
- new net: K3.1 (1~), Q1.4 (N)
- new net: K3.4, Q1.2
Changed lines of the file:
@@
 $EndDescr
-$Comp
-L Relay:FINDER-30.22 K3
-U 1 1 5F16ADE4
-P 5800 4300
-F 0 "K3" H 6430 4346 50  0000 L CNN
-F 1 "FINDER-30.22" H 6430 4255 50  0000 L CNN
-F 2 "Relay_THT:Relay_DPDT_Finder_30.22" H 7150 4270 50  0001 C CNN
-F 3 "http://gfinder.findernet.com/assets/Series/354/S30EN.pdf" H 5800 4300 50  0001 C CNN
-	1    5800 4300
-	1    0    0    -1
-$EndComp
 $Comp
 L MyParts:FI Q1
@@
 	0    1    1    0
 $EndComp
-Wire Wire Line
-	1200 1250 6100 1250
-Wire Wire Line
-	6100 1250 6100 4000
 Text HLabel 1200 1050 0    50   Input ~ 0
 230V_L
@@
 	1200 2050 3850 2050
 Wire Wire Line
-	5900 2050 5900 4000
-Wire Wire Line
 	1200 2250 3550 2250
-Wire Wire Line
-	5700 1050 10550 1050
-Connection ~ 5700 1050
-Wire Wire Line
-	6100 1250 10550 1250
-Connection ~ 6100 1250
 Wire Wire Line
 	1200 1450 2300 1450
@@
 	1200 1050 3300 1050
 Wire Wire Line
-	5400 4000 5400 2050
-Connection ~ 5400 2050
-Wire Wire Line
-	5400 2050 5900 2050
-Wire Wire Line
 	5400 4600 5400 4800
 Wire Wire Line
 	5400 4800 4950 4800
-Wire Wire Line
-	4950 4800 4950 2450
-Wire Wire Line
-	4400 2050 5400 2050
 Wire Wire Line
 	3850 2450 3550 2450
@@
 	3550 2450 3550 2250
 Wire Wire Line
-	4400 2450 4950 2450
-Connection ~ 4950 2450
-Wire Wire Line
-	4950 2450 6300 2450
-Wire Wire Line
-	6300 2450 6300 4000
-Wire Wire Line
-	3600 1050 5700 1050
-Wire Wire Line
-	5700 1050 5700 4000
+	3600 1050 5400 1050
 Wire Wire Line
 	6200 4600 6200 4800
@@
 Wire Wire Line
 	8950 2650 10550 2650
-Connection ~ 8950 1450
-Wire Wire Line
-	8950 1450 10550 1450
-Text HLabel 10550 1050 2    50   Input ~ 0
-230V_L_Out
-Text HLabel 10550 1250 2    50   Input ~ 0
-230V_N_Out
-Text HLabel 10550 1450 2    50   Input ~ 0
-230V_PE_Out
 Text HLabel 10550 2250 2    50   Input ~ 0
 230V_L_OutS
@@
 	1650 1950 1550 1950
 Wire Notes Line
-	10200 950  10300 950
-Wire Notes Line
-	10300 950  10300 1550
-Wire Notes Line
-	10300 1550 10200 1550
-Wire Notes Line
-	10200 1550 10200 950
-Wire Notes Line
 	10200 2150 10200 2750
 Wire Notes Line
@@
 Wire Notes Line
 	10300 2150 10200 2150
+Wire Wire Line
+	4400 2050 5700 2050
+Wire Wire Line
+	5400 4000 5400 1050
+Connection ~ 5400 1050
+Wire Wire Line
+	5400 1050 5900 1050
+Wire Wire Line
+	5700 4000 5700 2050
+$Comp
+L MyParts:FINDER-30.22 K3
+U 1 1 5F16ADE4
+P 5800 4300
+F 0 "K3" H 6430 4346 50  0000 L CNN
+F 1 "FINDER-30.22" H 6430 4255 50  0000 L CNN
+F 2 "Relay_THT:Relay_DPDT_Finder_30.22" H 7150 4270 50  0001 C CNN
+F 3 "http://gfinder.findernet.com/assets/Series/354/S30EN.pdf" H 5800 4300 50  0001 C CNN
+	1    5800 4300
+	1    0    0    -1
+$EndComp
+Wire Wire Line
+	5900 4000 5900 1050
+Wire Wire Line
+	1200 1250 4950 1250
+Wire Wire Line
+	6300 4000 6300 1250
+Wire Wire Line
+	4400 2450 6100 2450
+Wire Wire Line
+	4950 4800 4950 1250
+Connection ~ 4950 1250
+Wire Wire Line
+	4950 1250 6300 1250
+Wire Wire Line
+	6100 2450 6100 4000
 $EndSCHEMATC
