File: Schematics/12_PowerSupply.sch (KiCad schematic (older format))
At the start: 7 parts

Commit message: Finalize Schematic
Parts:
- removed U?: NAC3MPA-1-WOT, NAC3MPA-1-WOT, symbol BatteryBox-rescue:NAC3MPA-1-WOT-NAC3MPA-1-WOT
- added U2: VictronSmartSolarMppt7515, symbol MyParts:VictronSmartSolarMppt7515
- gave numbers to parts that had none: 6
Connections:
- net labels added: 0V_Cooler, 0V_Inverter, 0V_Panel, 0V_Relais, 12V_Charger_In, 12V_PowerSelector
- net labels removed: 0V_OUT, 12V+_OUT, 12V_Charger
- wire segments 20 -> 23
Other:
- note added: "Solar Panel"
Changed lines of the file:
@@
 Text HLabel 9450 4500 2    50   Input ~ 0
 0V_Charger
-Text HLabel 2300 2250 1    50   Input ~ 0
-12V+_OUT
-Text HLabel 2100 2450 1    50   Input ~ 0
-0V_OUT
 $Comp
 L Device:Battery BT?
@@
 P 7550 3600
 AR Path="/5F0C81D9/60D92067" Ref="BT?"  Part="1"
-AR Path="/60D529AB/60D84F6F/60D92067" Ref="BT?"  Part="1"
-F 0 "BT?" H 7658 3646 50  0000 L CNN
+AR Path="/60D529AB/60D84F6F/60D92067" Ref="BT1"  Part="1"
+F 0 "BT1" H 7658 3646 50  0000 L CNN
 F 1 "Battery" H 7658 3555 50  0000 L CNN
 F 2 "" V 7550 3660 50  0001 C CNN
@@
 $Comp
 L Switch:SW_DPST_x2 SW?
-U 2 1 60D9206D
+U 1 1 60D9206D
 P 7550 1700
 AR Path="/5F0C81D9/60D9206D" Ref="SW?"  Part="2"
-AR Path="/60D529AB/60D84F6F/60D9206D" Ref="SW?"  Part="2"
-F 0 "SW?" V 7596 1612 50  0000 R CNN
+AR Path="/60D529AB/60D84F6F/60D9206D" Ref="SW1"  Part="1"
+F 0 "SW1" V 7596 1612 50  0000 R CNN
 F 1 "SW_DPST_x2" V 7505 1612 50  0000 R CNN
 F 2 "" H 7550 1700 50  0001 C CNN
 F 3 "~" H 7550 1700 50  0001 C CNN
-	2    7550 1700
+	1    7550 1700
 	0    -1   -1   0
 $EndComp
@@
 P 4450 2050
 AR Path="/5F0C81D9/60D92073" Ref="U?"  Part="1"
-AR Path="/60D529AB/60D84F6F/60D92073" Ref="U?"  Part="1"
-F 0 "U?" H 4450 1227 50  0000 C CNN
+AR Path="/60D529AB/60D84F6F/60D92073" Ref="U3"  Part="1"
+F 0 "U3" H 4450 1227 50  0000 C CNN
 F 1 "F_Distributor" H 4450 1136 50  0000 C CNN
 F 2 "" H 4450 2050 50  0001 C CNN
 F 3 "" H 4450 2050 50  0001 C CNN
 	1    4450 2050
-	1    0    0    -1
-$EndComp
-$Comp
-L BatteryBox-rescue:NAC3MPA-1-WOT-NAC3MPA-1-WOT U?
-U 1 1 60D9207F
-P 1600 2650
-AR Path="/5F0C81D9/60D9207F" Ref="U?"  Part="1"
-AR Path="/60D529AB/60D84F6F/60D9207F" Ref="U?"  Part="1"
-F 0 "U?" H 1407 3417 50  0000 C CNN
-F 1 "NAC3MPA-1-WOT" H 1407 3326 50  0000 C CNN
-F 2 "NAC3MPA-1-WOT" H 1600 2650 50  0001 L BNN
-F 3 "" H 1600 2650 50  0001 C CNN
-	1    1600 2650
 	1    0    0    -1
 $EndComp
@@
 P 9000 4950
 AR Path="/5F0C81D9/60D920B5" Ref="X?"  Part="1"
-AR Path="/60D529AB/60D84F6F/60D920B5" Ref="X?"  Part="1"
-F 0 "X?" V 8145 4950 50  0000 C CNN
+AR Path="/60D529AB/60D84F6F/60D920B5" Ref="X1"  Part="1"
+F 0 "X1" V 8145 4950 50  0000 C CNN
 F 1 "Terminal16" V 8236 4950 50  0000 C CNN
 F 2 "MyParts:GroundTerminal" V 8327 4950 50  0000 C CNN
@@
 	7550 4500 7550 3800
 Wire Wire Line
-	1800 2250 3900 2250
-Wire Wire Line
-	8550 4800 3300 4800
-Wire Wire Line
-	3300 4800 3300 2450
-Wire Wire Line
-	3300 2450 1800 2450
-Wire Wire Line
 	7550 1100 7550 1500
 Wire Wire Line
@@
 P 7550 2650
 AR Path="/5F0C81D9/60D920D4" Ref="F?"  Part="1"
-AR Path="/60D529AB/60D84F6F/60D920D4" Ref="F?"  Part="1"
-F 0 "F?" H 7610 2696 50  0000 L CNN
+AR Path="/60D529AB/60D84F6F/60D920D4" Ref="F1"  Part="1"
+F 0 "F1" H 7610 2696 50  0000 L CNN
 F 1 "Fuse" H 7610 2605 50  0000 L CNN
 F 2 "" V 7480 2650 50  0001 C CNN
@@
 Wire Wire Line
 	7550 2800 7550 3400
-Text HLabel 5000 2250 2    50   Input ~ 0
-12V_Charger
+Text HLabel 3900 2650 0    50   Input ~ 0
+12V_Charger_In
 Wire Notes Line
 	7100 3250 8200 3250
@@
 P 1600 6050
 AR Path="/5F0C81D9/60D9D9F2" Ref="U?"  Part="1"
-AR Path="/60D529AB/60D84F6F/60D9D9F2" Ref="U?"  Part="1"
-F 0 "U?" H 1407 6817 50  0000 C CNN
+AR Path="/60D529AB/60D84F6F/60D9D9F2" Ref="U1"  Part="1"
+F 0 "U1" H 1407 6817 50  0000 C CNN
 F 1 "NAC3MPA-1-WOT" H 1407 6726 50  0000 C CNN
 F 2 "NAC3MPA-1-WOT" H 1600 6050 50  0001 L BNN
@@
 	1    0    0    -1
 $EndComp
-Wire Notes Line
-	3450 5650 5450 5600
-Wire Notes Line
-	5450 5600 5500 7000
-Wire Notes Line
-	5500 7000 3500 7000
-Wire Notes Line
-	3500 7000 3500 5650
-Wire Notes Line
-	3500 5650 4050 5400
-Wire Wire Line
-	5100 6000 4700 6000
-Wire Wire Line
-	5000 6300 8550 4900
-Wire Wire Line
-	1800 5650 3500 5850
-Wire Wire Line
-	1800 5850 3500 6100
 Wire Wire Line
 	4450 1100 7550 1100
+Text HLabel 5000 2650 2    50   Input ~ 0
+12V_Panel
+$Comp
+L MyParts:VictronSmartSolarMppt7515 U2
+U 1 1 60D65617
+P 4350 7200
+F 0 "U2" H 3772 6683 50  0000 R CNN
+F 1 "VictronSmartSolarMppt7515" H 3772 6774 50  0000 R CNN
+F 2 "" H 4350 7200 50  0001 C CNN
+F 3 "" H 4350 7200 50  0001 C CNN
+	1    4350 7200
+	-1   0    0    1
+$EndComp
 Wire Wire Line
-	4700 6000 3750 5150
+	3750 6400 3750 6050
 Wire Wire Line
-	3750 5150 3750 2450
+	4550 6400 4550 5200
 Wire Wire Line
-	3750 2450 3900 2450
-Text HLabel 5000 2450 2    50   Input ~ 0
-12V_Panel
+	4550 5200 8550 5200
+Wire Wire Line
+	4750 4000 4750 6400
+Wire Wire Line
+	4050 5650 1800 5650
+Wire Wire Line
+	4050 6400 4050 5650
+Wire Wire Line
+	3750 6050 9850 6050
+Wire Wire Line
+	1800 5850 4250 5850
+Wire Wire Line
+	4250 5850 4250 6400
+Text Notes 1200 5100 0    50   ~ 0
+Solar Panel
+Wire Notes Line
+	700  4800 2050 4800
+Wire Notes Line
+	2050 4800 2050 6700
+Wire Notes Line
+	2050 6700 700  6700
+Wire Notes Line
+	700  6700 700  4800
+Text HLabel 8550 4700 0    50   Input ~ 0
+0V_Inverter
+Text HLabel 8550 4800 0    50   Input ~ 0
+0V_Relais
+Text HLabel 8550 4900 0    50   Input ~ 0
+0V_Cooler
+Text HLabel 3900 2250 0    50   Input ~ 0
+12V_PowerSelector
+Text HLabel 8550 5000 0    50   Input ~ 0
+0V_Panel
+Wire Wire Line
+	9850 6050 9850 5100
+Wire Wire Line
+	9850 5100 9450 5100
+Wire Wire Line
+	3900 2450 3050 2450
+Wire Wire Line
+	3050 2450 3050 4000
+Wire Wire Line
+	3050 4000 4750 4000
 $EndSCHEMATC
