File: Schematics/Front_Panel.sch (KiCad schematic (older format))
At the start: 4 parts, among them J1 Conn_WallSocket, J2 Conn_WallSocket, SW1 SW_DPST_x2

Commit message: Finalize Schematic
Connections:
- net 0V renamed 0V_FrontPanel
- net 12V_In renamed 12V_In_FrontPanel
Changed lines of the file:
@@
 	1    0    0    -1
 $EndComp
-Connection ~ 3450 4100
-Text HLabel 1000 1100 0    50   Input ~ 0
-12V_In
-Text HLabel 1050 4100 0    50   Input ~ 0
-0V
+Connection ~ 3450 3650
+Text HLabel 1350 1100 0    50   Input ~ 0
+12V_In_FrontPanel
+Text HLabel 1400 3650 0    50   Input ~ 0
+0V_FrontPanel
 Wire Wire Line
-	1050 4100 3450 4100
+	1400 3650 3450 3650
 Wire Wire Line
-	1000 1100 1650 1100
+	1350 1100 1650 1100
 Wire Wire Line
 	2050 1100 3450 1100
@@
 	3450 1100 3450 2150
 Wire Wire Line
-	5900 2750 5900 4100
+	5900 2750 5900 3650
 Wire Wire Line
 	5900 1100 5900 2550
@@
 	3450 1100 5900 1100
 Wire Wire Line
-	3450 4100 5900 4100
+	3450 3650 5900 3650
 Wire Wire Line
 	3450 2150 4250 2150
@@
 	3450 2850 3450 3050
 Wire Wire Line
-	3450 3050 3450 4100
+	3450 3050 3450 3650
 Connection ~ 3450 3050
 Wire Notes Line
